File: usb_to_12v_bipolar_power.kicad_pcb (KiCad board)
At the start: 2 copper layers, 45.7 x 30.5 mm, 25 parts, among them J1 USB_A, J2 euro_power_header, J3 USB_5V_out, U1 CC3-0512DF-E

Commit message: add github link to pcb silkscreen
Other:
- board text added: "github.com/JordanAceto/ USB_to_bipolar_12VDC rev 1"
- board text removed: "Jordan Aceto USB to +-12V rev 1 2019-05-24"
Changed lines of the file:
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@@
   )
   (setup
-    (last_trace_width 1.016)
+    (last_trace_width 0.25)
     (user_trace_width 1.016)
     (trace_clearance 0.2)
@@
     )
   )
-  (gr_text "Jordan Aceto\nUSB to +-12V\nrev 1\n2019-05-24" (at 138.43 90.932) (layer B.SilkS)
+  (gr_text "github.com/JordanAceto/\nUSB_to_bipolar_12VDC\nrev 1" (at 138.176 89.916) (layer B.SilkS)
     (effects (font (size 1 1) (thickness 0.15)) (justify left mirror))
   )
